File: RFID_reader_v2.sch (EAGLE design)
At the start: 76 parts, among them IC1 78L05F, J1 PINOUT, U1 ESP-WROOM-32, U7 MFRC522, X1 CRYSTALS-NOGND-HC49/4H

Commit message: Add files via upload
Parts:
- removed J1: PINOUT, SparkFun-Connectors:CONN_08NO_SILK_FEMALE_PTH
- added A_TP1, A_TP2, A_TP3, MISO, MOSI, RST, RX_TP, RX_TP1, RX_TP2, SCK, SDA: (no value), pinhead:PINHD-1X1
- C16, C17, C29: value 0.1 uF -> 100n
- C18: value 100nF -> 100n
- C21, C23: value 180 pF -> 180p
- C22, C24: value 10 pF -> 10p
- C25, C28, C30, C31: value 15 pF -> 15p
- C26, C27: value 47 pF -> 47p
- C3: value 1nF -> 1n
- L2: value 15uH -> 15u
- L4, L5: value 2.2 uH -> 2.2u
- R19: value 10K -> 10k
- renumbered 12V_IN to GND_+12V, IC1 to 78L05, JP3 to RX_TX, L3 to L3_125K_ANT, U1 to ESP, U7 to MFRC522, X1 to 27.12MHZ
Connections:
- new net N$23: C17.1, RX_TP.1
- new net N$24: A_TP1.1, C21.1, C22.1, C25.2, RX_TP2.1
- new net N$25: A_TP3.1, C23.2, C24.2, C28.2
- net +3V3: no longer 78L05.VO, C32.+, J1.1
- net +5V: now also 78L05.VO, C32.+
- net GND: now also A_TP2.1; no longer C17.1, C21.1, C22.1, C23.2, C24.2, C25.2, C28.2, J1.3
- net IO13: no longer JP1.5
- net IO15: now also JP1.5
- net M-MFMISO: now also MISO.1; no longer J1.5
- net M-MFMOSI: now also MOSI.1; no longer J1.6
- net M-MFRST: now also RST.1; no longer J1.2
- net M-MFSCK: now also SCK.1; no longer J1.7
- net M-MFSDA: now also SDA.1; no longer J1.8
- net N$22: now also RX_TP1.1
Other:
- note added: "125kHz Antenna"
- note added: "12V to 3.3V Regulator"
- note added: "12V to 5V Regulator"
- note added: "ESP 32 Breakout"
- note added: "MFRC522 13.56MHz Reader"
- note removed: "12V Power Supply -> 5 V"
- note removed: "Antenna"
- moved on the sheet: C29
